File: hardware/Testapparaat/MCU.kicad_sch (KiCad schematic)
At the start: 9 parts

Commit message: -enh Made the schematic for the main unit almost complete :)
Parts:
- gave numbers to parts that had none: 9
Changed lines of the file:
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@@
   (symbol (lib_id "power:GND") (at 172.72 67.945 0) (unit 1)
     (in_bom yes) (on_board yes) (fields_autoplaced)
-    (property "Reference" "#PWR?" (id 0) (at 172.72 74.295 0)
+    (property "Reference" "#PWR027" (id 0) (at 172.72 74.295 0)
       (effects (font (size 1.27 1.27)) hide)
     )
@@
   (symbol (lib_id "Device:R") (at 58.42 154.305 90) (unit 1)
     (in_bom yes) (on_board yes) (fields_autoplaced)
-    (property "Reference" "R?" (id 0) (at 58.42 148.59 90))
+    (property "Reference" "R5" (id 0) (at 58.42 148.59 90))
     (property "Value" "10k" (id 1) (at 58.42 151.13 90))
     (property "Footprint" "" (id 2) (at 58.42 156.083 90)
@@
   (symbol (lib_id "RF_Module:ESP32-WROOM-32") (at 95.25 76.2 0) (unit 1)
     (in_bom yes) (on_board yes) (fields_autoplaced)
-    (property "Reference" "U?" (id 0) (at 97.2694 38.1 0)
+    (property "Reference" "U2" (id 0) (at 97.2694 38.1 0)
       (effects (font (size 1.27 1.27)) (justify left))
     )
@@
   (symbol (lib_id "Switch:SW_Push") (at 34.925 29.845 0) (unit 1)
     (in_bom yes) (on_board yes) (fields_autoplaced)
-    (property "Reference" "SW?" (id 0) (at 34.925 21.59 0))
+    (property "Reference" "SW1" (id 0) (at 34.925 21.59 0))
     (property "Value" "RST" (id 1) (at 34.925 24.13 0))
     (property "Footprint" "" (id 2) (at 34.925 24.765 0)
@@
   (symbol (lib_id "Connector_Generic:Conn_02x06_Odd_Even") (at 177.8 60.325 0) (unit 1)
     (in_bom yes) (on_board yes) (fields_autoplaced)
-    (property "Reference" "J?" (id 0) (at 179.07 48.26 0))
+    (property "Reference" "J4" (id 0) (at 179.07 48.26 0))
     (property "Value" "DEBUG" (id 1) (at 179.07 50.8 0))
     (property "Footprint" "" (id 2) (at 177.8 60.325 0)
@@
   (symbol (lib_id "Device:R") (at 40.64 26.035 0) (unit 1)
     (in_bom yes) (on_board yes) (fields_autoplaced)
-    (property "Reference" "R?" (id 0) (at 43.18 24.7649 0)
+    (property "Reference" "R3" (id 0) (at 43.18 24.7649 0)
       (effects (font (size 1.27 1.27)) (justify left))
     )
@@
   (symbol (lib_id "power:+3.3V") (at 189.865 55.245 270) (unit 1)
     (in_bom yes) (on_board yes) (fields_autoplaced)
-    (property "Reference" "#PWR?" (id 0) (at 186.055 55.245 0)
+    (property "Reference" "#PWR028" (id 0) (at 186.055 55.245 0)
       (effects (font (size 1.27 1.27)) hide)
     )
@@
   (symbol (lib_id "Transistor_BJT:BC817") (at 67.31 154.305 0) (mirror x) (unit 1)
     (in_bom yes) (on_board yes) (fields_autoplaced)
-    (property "Reference" "Q?" (id 0) (at 72.39 153.0349 0)
+    (property "Reference" "Q2" (id 0) (at 72.39 153.0349 0)
       (effects (font (size 1.27 1.27)) (justify left))
     )
@@
   (symbol (lib_id "power:+3.3V") (at 40.64 22.225 0) (unit 1)
     (in_bom yes) (on_board yes) (fields_autoplaced)
-    (property "Reference" "#PWR?" (id 0) (at 40.64 26.035 0)
+    (property "Reference" "#PWR023" (id 0) (at 40.64 26.035 0)
       (effects (font (size 1.27 1.27)) hide)
     )
@@
   (symbol (lib_id "power:+3.3V") (at 95.25 40.64 0) (unit 1)
     (in_bom yes) (on_board yes) (fields_autoplaced)
-    (property "Reference" "#PWR?" (id 0) (at 95.25 44.45 0)
+    (property "Reference" "#PWR025" (id 0) (at 95.25 44.45 0)
       (effects (font (size 1.27 1.27)) hide)
     )
@@
   (symbol (lib_id "power:GND") (at 29.845 29.845 0) (unit 1)
     (in_bom yes) (on_board yes) (fields_autoplaced)
-    (property "Reference" "#PWR?" (id 0) (at 29.845 36.195 0)
+    (property "Reference" "#PWR022" (id 0) (at 29.845 36.195 0)
       (effects (font (size 1.27 1.27)) hide)
     )
@@
   (symbol (lib_id "Device:C") (at 40.64 33.655 0) (unit 1)
     (in_bom yes) (on_board yes) (fields_autoplaced)
-    (property "Reference" "C?" (id 0) (at 44.45 32.3849 0)
+    (property "Reference" "C1" (id 0) (at 44.45 32.3849 0)
       (effects (font (size 1.27 1.27)) (justify left))
     )
@@
   (symbol (lib_id "power:GND") (at 95.25 111.76 0) (unit 1)
     (in_bom yes) (on_board yes) (fields_autoplaced)
-    (property "Reference" "#PWR?" (id 0) (at 95.25 118.11 0)
+    (property "Reference" "#PWR026" (id 0) (at 95.25 118.11 0)
       (effects (font (size 1.27 1.27)) hide)
     )
@@
   (symbol (lib_id "Device:R") (at 58.42 139.7 90) (unit 1)
     (in_bom yes) (on_board yes) (fields_autoplaced)
-    (property "Reference" "R?" (id 0) (at 58.42 133.985 90))
+    (property "Reference" "R4" (id 0) (at 58.42 133.985 90))
     (property "Value" "10k" (id 1) (at 58.42 136.525 90))
     (property "Footprint" "" (id 2) (at 58.42 141.478 90)
@@
   (symbol (lib_id "Transistor_BJT:BC817") (at 67.31 139.7 0) (unit 1)
     (in_bom yes) (on_board yes) (fields_autoplaced)
-    (property "Reference" "Q?" (id 0) (at 72.39 138.4299 0)
+    (property "Reference" "Q1" (id 0) (at 72.39 138.4299 0)
       (effects (font (size 1.27 1.27)) (justify left))
     )
@@
   (symbol (lib_id "power:GND") (at 40.64 37.465 0) (unit 1)
     (in_bom yes) (on_board yes) (fields_autoplaced)
-    (property "Reference" "#PWR?" (id 0) (at 40.64 43.815 0)
-      (effects (font (size 1.27 1.27)) hide)
-    )
+    (property "Reference" "#PWR024" (id 0) (at 40.64 43.815 0)
+      (effects (font (size 1.27 1.27)) hide)
+    )

Commit message: -enh made some changes to schematic and assigned fp
Parts:
- C1: footprint (none) -> Capacitor_SMD:C_0603_1608Metric_Pad1.08x0.95mm_HandSolder
- J4: footprint (none) -> Connector_PinHeader_2.54mm:PinHeader_2x06_P2.54mm_Vertical_SMD
- R3, R4, R5: footprint (none) -> Resistor_SMD:R_0603_1608Metric_Pad0.98x0.95mm_HandSolder
- SW1: footprint (none) -> Button_Switch_SMD:SW_SPST_B3S-1000
Changed lines of the file:
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@@
     (property "Reference" "R5" (id 0) (at 58.42 148.59 90))
     (property "Value" "10k" (id 1) (at 58.42 151.13 90))
-    (property "Footprint" "" (id 2) (at 58.42 156.083 90)
+    (property "Footprint" "Resistor_SMD:R_0603_1608Metric_Pad0.98x0.95mm_HandSolder" (id 2) (at 58.42 156.083 90)
       (effects (font (size 1.27 1.27)) hide)
     )
@@
     (property "Reference" "SW1" (id 0) (at 34.925 21.59 0))
     (property "Value" "RST" (id 1) (at 34.925 24.13 0))
-    (property "Footprint" "" (id 2) (at 34.925 24.765 0)
+    (property "Footprint" "Button_Switch_SMD:SW_SPST_B3S-1000" (id 2) (at 34.925 24.765 0)
       (effects (font (size 1.27 1.27)) hide)
     )
@@
     (property "Reference" "J4" (id 0) (at 179.07 48.26 0))
     (property "Value" "DEBUG" (id 1) (at 179.07 50.8 0))
-    (property "Footprint" "" (id 2) (at 177.8 60.325 0)
+    (property "Footprint" "Connector_PinHeader_2.54mm:PinHeader_2x06_P2.54mm_Vertical_SMD" (id 2) (at 177.8 60.325 0)
       (effects (font (size 1.27 1.27)) hide)
     )
@@
       (effects (font (size 1.27 1.27)) (justify left))
     )
-    (property "Footprint" "" (id 2) (at 38.862 26.035 90)
+    (property "Footprint" "Resistor_SMD:R_0603_1608Metric_Pad0.98x0.95mm_HandSolder" (id 2) (at 38.862 26.035 90)
       (effects (font (size 1.27 1.27)) hide)
     )
@@
       (effects (font (size 1.27 1.27)) (justify left))
     )
-    (property "Footprint" "" (id 2) (at 41.6052 37.465 0)
+    (property "Footprint" "Capacitor_SMD:C_0603_1608Metric_Pad1.08x0.95mm_HandSolder" (id 2) (at 41.6052 37.465 0)
       (effects (font (size 1.27 1.27)) hide)
     )
@@
     (property "Reference" "R4" (id 0) (at 58.42 133.985 90))
     (property "Value" "10k" (id 1) (at 58.42 136.525 90))
-    (property "Footprint" "" (id 2) (at 58.42 141.478 90)
-      (effects (font (size 1.27 1.27)) hide)
-    )
+    (property "Footprint" "Resistor_SMD:R_0603_1608Metric_Pad0.98x0.95mm_HandSolder" (id 2) (at 58.42 141.478 90)
+      (effects (font (size 1.27 1.27)) hide)
+    )

Commit message: -add BOM
Parts:
- added C13: 100n, Capacitor_SMD:C_0603_1608Metric_Pad1.08x0.95mm_HandSolder, symbol Device:C_Small
Connections:
- net +3.3V: now also C13.1
- net GND: now also C13.2
Changed lines of the file:
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@@
 (kicad_sch (version 20211123) (generator eeschema)
   (paper "A4")
+  (junction (at 95.25 32.004) (diameter 0) (color 0 0 0 0)
+  )
   (junction (at 40.64 29.845) (diameter 0) (color 0 0 0 0)
   )
@@
     (stroke (width 0) (type default) (color 0 0 0 0))
   )
+  (wire (pts (xy 89.662 32.004) (xy 95.25 32.004))
+    (stroke (width 0) (type default) (color 0 0 0 0))
+  )
   (wire (pts (xy 54.61 147.32) (xy 69.85 147.32))
     (stroke (width 0) (type default) (color 0 0 0 0))
@@
     (stroke (width 0) (type default) (color 0 0 0 0))
   )
+  (wire (pts (xy 95.25 31.496) (xy 95.25 32.004))
+    (stroke (width 0) (type default) (color 0 0 0 0))
+  )
   (wire (pts (xy 69.85 132.715) (xy 69.85 134.62))
+    (stroke (width 0) (type default) (color 0 0 0 0))
+  )
+  (wire (pts (xy 95.25 32.004) (xy 95.25 40.64))
     (stroke (width 0) (type default) (color 0 0 0 0))
   )
@@
     (pin "9")
   )
+  (symbol (lib_id "Device:C_Small") (at 89.662 34.544 0) (unit 1)
+    (in_bom yes) (on_board yes)
+    (property "Reference" "C13" (id 0) (at 84.836 33.274 0)
+      (effects (font (size 1.27 1.27)) (justify left))
+    )
+    (property "Value" "100n" (id 1) (at 83.566 36.068 0)
+      (effects (font (size 1.27 1.27)) (justify left))
+    )
+    (property "Footprint" "Capacitor_SMD:C_0603_1608Metric_Pad1.08x0.95mm_HandSolder" (id 2) (at 89.662 34.544 0)
+      (effects (font (size 1.27 1.27)) hide)
+    )
+    (property "Datasheet" "~" (id 3) (at 89.662 34.544 0)
+      (effects (font (size 1.27 1.27)) hide)
+    )
+    (pin "1")
+    (pin "2")
+  )
+  (symbol (lib_id "power:GND") (at 89.662 37.084 0) (unit 1)
+    (in_bom yes) (on_board yes) (fields_autoplaced)
+    (property "Reference" "#PWR0101" (id 0) (at 89.662 43.434 0)
+      (effects (font (size 1.27 1.27)) hide)
+    )
+    (property "Value" "GND" (id 1) (at 89.662 41.529 0))
+    (property "Footprint" "" (id 2) (at 89.662 37.084 0)
+      (effects (font (size 1.27 1.27)) hide)
+    )
+    (property "Datasheet" "" (id 3) (at 89.662 37.084 0)
+      (effects (font (size 1.27 1.27)) hide)
+    )
+    (pin "1")
+  )
   (symbol (lib_id "Switch:SW_Push") (at 34.925 29.845 0) (unit 1)
     (in_bom yes) (on_board yes) (fields_autoplaced)
@@
     (pin "1")
   )
-  (symbol (lib_id "power:+3.3V") (at 95.25 40.64 0) (unit 1)
-    (in_bom yes) (on_board yes) (fields_autoplaced)
-    (property "Reference" "#PWR025" (id 0) (at 95.25 44.45 0)
-      (effects (font (size 1.27 1.27)) hide)
-    )
-    (property "Value" "+3.3V" (id 1) (at 95.25 35.56 0))
-    (property "Footprint" "" (id 2) (at 95.25 40.64 0)
-      (effects (font (size 1.27 1.27)) hide)
-    )
-    (property "Datasheet" "" (id 3) (at 95.25 40.64 0)
-      (effects (font (size 1.27 1.27)) hide)
-    )
+  (symbol (lib_id "power:+3.3V") (at 95.25 31.496 0) (unit 1)
+    (in_bom yes) (on_board yes) (fields_autoplaced)
+    (property "Reference" "#PWR025" (id 0) (at 95.25 35.306 0)
+      (effects (font (size 1.27 1.27)) hide)
+    )
+    (property "Value" "+3.3V" (id 1) (at 95.25 26.416 0))
+    (property "Footprint" "" (id 2) (at 95.25 31.496 0)
+      (effects (font (size 1.27 1.27)) hide)
+    )
+    (property "Datasheet" "" (id 3) (at 95.25 31.496 0)
+      (effects (font (size 1.27 1.27)) hide)
+    )

Commit message: -enh Made a start at pcb design
Connections:
- net DTS is gone; now on net DTR: J4.9 (Pin_9)
Changed lines of the file:
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@@
     )
   )
-  (global_label "DTS" (shape input) (at 172.72 65.405 180) (fields_autoplaced)
+  (global_label "DTR" (shape input) (at 172.72 65.405 180) (fields_autoplaced)
     (effects (font (size 1.27 1.27)) (justify right))
-    (property "Intersheet-verwijzingen" "${INTERSHEET_REFS}" (id 0) (at 166.8598 65.3256 0)
+    (property "Intersheet-verwijzingen" "${INTERSHEET_REFS}" (id 0) (at 166.7993 65.3256 0)
       (effects (font (size 1.27 1.27)) (justify right) hide)
     )
