File: hardware/Testapparaat/Testapparaat.kicad_pcb (KiCad board)
At the start: 2 copper layers, 127 x 142.2 mm, 107 parts, among them J1 IO_SD, J10 B-, J11 Display_shield, J12 GPIO_INPUTS, J13 FrontPanel, J14 GPIO_OUTPUT, J2 Module_1, J3 Module_2, J4 DEBUG, J5 FPC_40P_LCD_ILI9488, J6 IO_UART, J7 Emergency Stop Button, J8 CON-SOCJ-2155, J9 B+, Q1 BC817, Q2 BC817, Q3 BC817, Q4 IRFR9024N, Q5 IRFR9024N, Q6 IRFR9024N, SW1 RST, SW2 on/off switch, U1 74HC595 (SIPO Shift register), U10 LM2596S-5, U11 LM2596S-3.3, U12 74AUC1G74, U2 ESP32-WROOM-32, U4 74HC595 (SIPO Shift register), U5 TCA9534 (IO Expander), U6 74HC14, U7 TCA9534 (IO Expander), U8 74HC14, U9 74HC14

Commit message: -enh Routed everything
Parts:
- C15: moved to F.Cu
- moved C16 82.8 mm to (163.7, 42.1)
- moved R33 38.7 mm to (137.0, 96.2), turned to 0 degrees
- moved D3 35.2 mm to (136.9, 98.0), turned to 180 degrees
- moved R7 33.3 mm to (190.0, 154.3), turned to 180 degrees
- moved C15 33.2 mm to (118.8, 129.8), turned to -90 degrees
- moved R8 32.8 mm to (186.9, 154.3), turned to 180 degrees
- moved C1 30.2 mm to (140.3, 62.4)
- moved R3 20.1 mm to (136.7, 62.6), turned to 0 degrees
- moved R14 14.7 mm to (127.8, 121.5), turned to -90 degrees
- moved SW2 13.8 mm to (229.5, 133.4)
- moved C3 13.6 mm to (224.4, 136.3)
- moved R6 13.6 mm to (226.1, 136.4)
- moved R15 12.9 mm to (125.4, 121.5), turned to -90 degrees
- moved J8 11.1 mm to (227.3, 147.2)
- moved C10 6.54 mm to (122.7, 127.5), turned to -90 degrees
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Routing:
- net +3.3V: track 348.7 -> 592.6 mm, vias 13 -> 26
- net GND: track 43.2 -> 199.3 mm, vias 11 -> 41
- net MOD_PSU_EN: track 0.00 -> 151.5 mm, vias 0 -> 4
- net REG_EN: track 5.02 -> 116.7 mm, vias 0 -> 2
- net EMERGENCY_STOP_BTN: track 2.77 -> 91.3 mm, vias 0 -> 6
- net GPIO_INPUT_1: track 0.00 -> 62.6 mm, vias 0 -> 3
- net Rotary_BTN: track 0.00 -> 60.4 mm, vias 0 -> 3
- net GPIO_INPUT_2: track 1.74 -> 50.6 mm
- net Net-(C21-Pad1): track 0.00 -> 47.8 mm, vias 0 -> 2
- net +5V: track 165.9 -> 211.6 mm
- net BTN_1: track 0.00 -> 40.8 mm, vias 0 -> 1
- net BTN_2: track 0.00 -> 38.8 mm, vias 0 -> 1
- net BTN_4: track 0.00 -> 34.4 mm, vias 0 -> 1
- net BTN_8: track 0.00 -> 33.8 mm, vias 0 -> 1
- net BTN_6: track 0.00 -> 32.9 mm, vias 0 -> 1
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Other:
- board size 127 x 142.2 mm -> 138.1 x 142.2 mm
