File: hardware/Testapparaat/Testapparaat.kicad_sch (KiCad schematic)
At the start: 33 parts, among them J1 IO_SD, J14 GPIO_OUTPUT, J2 Module_1, J3 Module_2, J6 IO_UART, J7 Emergency Stop Button, Q3 BC817, Q4 IRFR9024N, Q5 IRFR9024N, Q6 IRFR9024N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

Commit message: -enh Final adjustments
Connections:
- net GPIO_INPUT_1 renamed Display_TP_IRQ
Other:
- sheet Display ports: added Display_TP_IRQ, SPI_MISO; removed none
Changed lines of the file:
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@@
+    (stroke (width 0) (type default) (color 0 0 0 0))
+  )
+  (wire (pts (xy 76.2 45.974) (xy 73.66 45.974))
     (stroke (width 0) (type default) (color 0 0 0 0))
   )
@@
     )
   )
+  (global_label "Display_TP_IRQ" (shape input) (at 265.43 67.056 0) (fields_autoplaced)
+    (effects (font (size 1.27 1.27)) (justify left))
+    (property "Intersheet References" "${INTERSHEET_REFS}" (id 0) (at 282.055 66.9766 0)
+      (effects (font (size 1.27 1.27)) (justify left) hide)
+    )
+  )
   (global_label "SPI_MISO" (shape input) (at 42.926 55.88 0) (fields_autoplaced)
     (effects (font (size 1.27 1.27)) (justify left))
@@
     )
   )
+  (global_label "SPI_MISO" (shape input) (at 73.66 49.53 0) (fields_autoplaced)
+    (effects (font (size 1.27 1.27)) (justify left))
+    (property "Intersheet-verwijzingen" "${INTERSHEET_REFS}" (id 0) (at 84.7212 49.4506 0)
+      (effects (font (size 1.27 1.27)) (justify left) hide)
+    )
+  )
   (global_label "TTL2_MOD_2" (shape input) (at 153.67 90.678 0) (fields_autoplaced)
     (effects (font (size 1.27 1.27)) (justify left))
@@
     (effects (font (size 1.27 1.27)) (justify left))
     (property "Intersheet-verwijzingen" "${INTERSHEET_REFS}" (id 0) (at 118.5758 117.0146 0)
-      (effects (font (size 1.27 1.27)) (justify left) hide)
-    )
-  )
-  (global_label "GPIO_INPUT_1" (shape input) (at 265.43 67.056 0) (fields_autoplaced)
-    (effects (font (size 1.27 1.27)) (justify left))
-    (property "Intersheet-verwijzingen" "${INTERSHEET_REFS}" (id 0) (at 280.9664 66.9766 0)
       (effects (font (size 1.27 1.27)) (justify left) hide)
     )
@@
     (property "Intersheet-verwijzingen" "${INTERSHEET_REFS}" (id 0) (at 49.8988 102.5366 0)
       (effects (font (size 1.27 1.27)) (justify right) hide)
+    )
+  )
+  (global_label "Display_TP_IRQ" (shape output) (at 76.2 45.974 0) (fields_autoplaced)
+    (effects (font (size 1.27 1.27)) (justify left))
+    (property "Intersheet References" "${INTERSHEET_REFS}" (id 0) (at 92.825 45.8946 0)
+      (effects (font (size 1.27 1.27)) (justify left) hide)
     )
   )
@@
       (effects (font (size 1.27 1.27)) (justify left))
     )
+    (pin "Display_TP_IRQ" input (at 73.66 45.974 0)
+      (effects (font (size 1.27 1.27)) (justify right))
+    )
+    (pin "SPI_MISO" input (at 73.66 49.53 0)
+      (effects (font (size 1.27 1.27)) (justify right))
+    )
   )
   (sheet_instances
@@
       (reference "#PWR038") (unit 1) (value "GND") (footprint "")
     )
-    (path "/20b97c1c-ceb0-4084-b6e4-51876929be6d/343548c1-7a9b-4798-8a8d-b474ba77e7d0"
-      (reference "#PWR039") (unit 1) (value "GND") (footprint "")
-    )
-    (path "/20b97c1c-ceb0-4084-b6e4-51876929be6d/24f07e2b-0af1-4d37-b546-aac23a0e38f1"
-      (reference "#PWR040") (unit 1) (value "+3.3V") (footprint "")
-    )
     (path "/20b97c1c-ceb0-4084-b6e4-51876929be6d/076b870d-ede1-4533-8bbb-b96819d335d1"
       (reference "#PWR041") (unit 1) (value "+3.3V") (footprint "")
@@
       (reference "J11") (unit 1) (value "Display_shield") (footprint "Connector_PinHeader_2.54mm:PinHeader_2x13_P2.54mm_Vertical_SMD")
     )
-    (path "/20b97c1c-ceb0-4084-b6e4-51876929be6d/a24376a2-6ff7-4689-b696-69bccae7fcd8"
-      (reference "J12") (unit 1) (value "GPIO_INPUTS") (footprint "Connector_PinHeader_2.54mm:PinHeader_1x04_P2.54mm_Horizontal")
-    )
     (path "/20b97c1c-ceb0-4084-b6e4-51876929be6d/33557b62-dd40-4840-8a8d-47b10828cc23"
