File: hardware/Testapparaat/button_inputs.kicad_sch (KiCad schematic)
At the start: 25 parts, among them J12 GPIO_INPUTS, J13 FrontPanel, U6 74HC14, U8 74HC14, U9 74HC14

Commit message: -enh Made a start at pcb design
Parts:
- added C4, C5, C7: 1u, Capacitor_SMD:C_0603_1608Metric_Pad1.08x0.95mm_HandSolder, symbol Device:C
- added D5, D6, D7: 1N4448WS, Diode_SMD:D_SOD-323, symbol Diode:1N4448WS
- added R42, R43, R44: 10k, Resistor_SMD:R_0603_1608Metric_Pad0.98x0.95mm_HandSolder, symbol Device:R
- added U12: 74AUC1G74, Package_SO:VSSOP-8_2.3x2mm_P0.5mm, symbol 74xGxx:74AUC1G74
Connections:
- net +3.3V: now also U12.6 (~{CLR}), U12.7 (~{PRE}), U12.8 (VCC)
- net GND: now also C4.2, C5.2, C7.2, U12.4 (GND)
- net Rotary_BTN_R: now also D7.2 (A), R44.1; no longer R34.2, U9.3
- net Rotary_CLK: now also U12.1 (C)
- net Rotary_CLK_R: now also J13.12 (Pin_12), D6.2 (A), R43.1; no longer J13.14 (Pin_14), R29.2, U9.1
- net Rotary_DT: now also U12.5 (Q); no longer U9.6
- net Rotary_DT_R: no longer names the net of R35.2, U9.5
- net Rotary_DT_R: now also C4.1, D5.1 (K), R42.2; no longer J13.12 (Pin_12)
- new net: C5.1, D6.1 (K), R29.2, R43.2, U9.1
- new net: C7.1, D7.1 (K), R34.2, R44.2, U9.3
- new net Rotary_B: U12.2 (D), U9.6
- new net Rotary_B_R: D5.2 (A), J13.14 (Pin_14), R42.1
- no-connect marks 3 -> 4

Commit message: -add gerbers and minor improvements
Connections:
- net GPIO_INPUT_2_R: no longer R27.2, U9.11
- net GPIO_INPUT_2: no longer names the net of U9.10
- new net: R27.2, U9.11
- no-connect marks 4 -> 5
Changed lines of the file:
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@@
   (junction (at 60.96 43.688) (diameter 0) (color 0 0 0 0)
-  )
-  (junction (at 170.434 75.946) (diameter 0) (color 0 0 0 0)
   )
   (junction (at 170.942 32.004) (diameter 0) (color 0 0 0 0)
@@
   (no_connect (at 42.164 103.886))
   (no_connect (at 159.258 119.888))
+  (no_connect (at 155.194 75.946))
   (no_connect (at 155.448 87.376))
   (no_connect (at 97.536 86.106))
@@
     (stroke (width 0) (type default) (color 0 0 0 0))
   )
-  (wire (pts (xy 170.434 75.946) (xy 181.102 75.946))
-    (stroke (width 0) (type default) (color 0 0 0 0))
-  )
   (wire (pts (xy 112.776 80.518) (xy 112.776 81.026))
     (stroke (width 0) (type default) (color 0 0 0 0))
@@
     )
   )
-  (global_label "GPIO_INPUT_2" (shape input) (at 155.194 75.946 180) (fields_autoplaced)
-    (effects (font (size 1.27 1.27)) (justify right))
-    (property "Intersheet-verwijzingen" "${INTERSHEET_REFS}" (id 0) (at 139.6576 75.8666 0)
-      (effects (font (size 1.27 1.27)) (justify right) hide)
-    )
-  )
   (global_label "BTN_10" (shape output) (at 97.282 74.422 180) (fields_autoplaced)
     (effects (font (size 1.27 1.27)) (justify right))
@@
       (effects (font (size 1.27 1.27)) (justify left) hide)
     )
-  )
-  (global_label "GPIO_INPUT_2_R" (shape input) (at 181.102 75.946 0) (fields_autoplaced)
-    (effects (font (size 1.27 1.27)) (justify left))
-    (property "Intersheet-verwijzingen" "${INTERSHEET_REFS}" (id 0) (at 198.8761 75.8666 0)
-      (effects (font (size 1.27 1.27)) (justify left) hide)
-    )

Commit message: -enh Final adjustments
Parts:
- removed J12: GPIO_INPUTS, Connector_PinHeader_2.54mm:PinHeader_1x04_P2.54mm_Horizontal, symbol Connector:Conn_01x04_Male
Connections:
- net GPIO_INPUT_1: no longer names the net of U9.8
- net GPIO_INPUT_1_R: no longer names the net of R26.2, U9.9
- no-connect marks 5 -> 6
Changed lines of the file:
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@@
   (junction (at 112.522 53.34) (diameter 0) (color 0 0 0 0)
   )
-  (junction (at 170.434 65.024) (diameter 0) (color 0 0 0 0)
-  )
   (junction (at 184.912 53.848) (diameter 0) (color 0 0 0 0)
   )
@@
   )
   (no_connect (at 42.164 103.886))
+  (no_connect (at 155.194 65.024))
   (no_connect (at 159.258 119.888))
   (no_connect (at 155.194 75.946))
@@
     (stroke (width 0) (type default) (color 0 0 0 0))
   )
-  (wire (pts (xy 53.34 133.604) (xy 53.34 135.89))
-    (stroke (width 0) (type default) (color 0 0 0 0))
-  )
-  (wire (pts (xy 170.434 65.024) (xy 181.102 65.024))
-    (stroke (width 0) (type default) (color 0 0 0 0))
-  )
   (wire (pts (xy 230.378 25.908) (xy 230.378 29.718))
     (stroke (width 0) (type default) (color 0 0 0 0))
@@
     (stroke (width 0) (type default) (color 0 0 0 0))
   )
-  (wire (pts (xy 53.34 135.89) (xy 47.498 135.89))
-    (stroke (width 0) (type default) (color 0 0 0 0))
-  )
   (wire (pts (xy 193.802 35.306) (xy 193.802 37.338))
     (stroke (width 0) (type default) (color 0 0 0 0))
@@
     (stroke (width 0) (type default) (color 0 0 0 0))
   )
-  (global_label "GPIO_INPUT_1" (shape input) (at 155.194 65.024 180) (fields_autoplaced)
-    (effects (font (size 1.27 1.27)) (justify right))
-    (property "Intersheet-verwijzingen" "${INTERSHEET_REFS}" (id 0) (at 139.6576 64.9446 0)
-      (effects (font (size 1.27 1.27)) (justify right) hide)
-    )
-  )
   (global_label "BTN_9_R" (shape output) (at 54.864 111.506 0) (fields_autoplaced)
     (effects (font (size 1.27 1.27)) (justify left))
@@
     )
   )
-  (global_label "GPIO_INPUT_1_R" (shape input) (at 181.102 65.024 0) (fields_autoplaced)
-    (effects (font (size 1.27 1.27)) (justify left))
-    (property "Intersheet-verwijzingen" "${INTERSHEET_REFS}" (id 0) (at 198.8761 64.9446 0)
-      (effects (font (size 1.27 1.27)) (justify left) hide)
-    )
-  )
   (global_label "BTN_2_R" (shape input) (at 70.612 43.688 0) (fields_autoplaced)
     (effects (font (size 1.27 1.27)) (justify left))
@@
     (property "Intersheet-verwijzingen" "${INTERSHEET_REFS}" (id 0) (at 31.768 116.5066 0)
       (effects (font (size 1.27 1.27)) (justify right) hide)
-    )
-  )
-  (global_label "GPIO_INPUT_2_R" (shape input) (at 47.498 140.97 0) (fields_autoplaced)
-    (effects (font (size 1.27 1.27)) (justify left))
-    (property "Intersheet-verwijzingen" "${INTERSHEET_REFS}" (id 0) (at 65.2721 140.8906 0)
-      (effects (font (size 1.27 1.27)) (justify left) hide)
-    )
-  )
-  (global_label "GPIO_INPUT_1_R" (shape input) (at 47.498 138.43 0) (fields_autoplaced)
-    (effects (font (size 1.27 1.27)) (justify left))
-    (property "Intersheet-verwijzingen" "${INTERSHEET_REFS}" (id 0) (at 65.2721 138.3506 0)
-      (effects (font (size 1.27 1.27)) (justify left) hide)
     )
   )
@@
     (pin "1")
     (pin "2")
-  )
-  (symbol (lib_id "power:+3.3V") (at 53.34 133.604 0) (unit 1)
-    (in_bom yes) (on_board yes) (fields_autoplaced)
-    (property "Reference" "#PWR040" (id 0) (at 53.34 137.414 0)
-      (effects (font (size 1.27 1.27)) hide)
-    )
-    (property "Value" "+3.3V" (id 1) (at 53.34 130.0282 0))
-    (property "Footprint" "" (id 2) (at 53.34 133.604 0)
-      (effects (font (size 1.27 1.27)) hide)
-    )
-    (property "Datasheet" "" (id 3) (at 53.34 133.604 0)
-      (effects (font (size 1.27 1.27)) hide)
-    )
-    (pin "1")
   )
   (symbol (lib_id "power:+3.3V") (at 170.688 82.296 0) (unit 1)
@@
     (pin "2")
   )
-  (symbol (lib_id "power:GND") (at 47.498 143.51 0) (unit 1)
-    (in_bom yes) (on_board yes) (fields_autoplaced)
-    (property "Reference" "#PWR039" (id 0) (at 47.498 149.86 0)
-      (effects (font (size 1.27 1.27)) hide)
-    )
-    (property "Value" "GND" (id 1) (at 47.498 147.9534 0))
-    (property "Footprint" "" (id 2) (at 47.498 143.51 0)
-      (effects (font (size 1.27 1.27)) hide)
-    )
-    (property "Datasheet" "" (id 3) (at 47.498 143.51 0)
-      (effects (font (size 1.27 1.27)) hide)
-    )
-    (pin "1")
-  )
   (symbol (lib_id "74xx:74HC14") (at 105.156 86.106 180) (unit 6)
     (in_bom yes) (on_board yes)
@@
     (pin "7")
   )
-  (symbol (lib_id "Connector:Conn_01x04_Male") (at 42.418 138.43 0) (unit 1)
-    (in_bom yes) (on_board yes)
-    (property "Reference" "J12" (id 0) (at 45.72 130.81 0))
-    (property "Value" "GPIO_INPUTS" (id 1) (at 46.228 133.096 0))
-    (property "Footprint" "Connector_PinHeader_2.54mm:PinHeader_1x04_P2.54mm_Horizontal" (id 2) (at 42.418 138.43 0)
-      (effects (font (size 1.27 1.27)) hide)
-    )
-    (property "Datasheet" "~" (id 3) (at 42.418 138.43 0)
-      (effects (font (size 1.27 1.27)) hide)
-    )
-    (pin "1")
-    (pin "2")
-    (pin "3")
-    (pin "4")
-  )
   (symbol (lib_id "power:GND") (at 230.886 103.124 0) (unit 1)
