File: hardware/Testapparaat_IO/Testapparaat_io/Testapparaat_io.kicad_pcb (KiCad board)
At the start: 2 copper layers, 34.5 x 65.8 mm, 15 parts, among them J1 IO_UART, J2 IO_SD, J3 MEM2051-00-195-00-A, J4 DB9_Female, U1 MAX3232

Commit message: -add gerbers of IO pcb
Parts:
- moved REF** 1.64 mm to (125.0, 34.1)
- moved REF** 0.72 mm to (152.2, 93.5)
- moved REF** 0.69 mm to (124.3, 93.6)
- moved REF** 0.65 mm to (151.9, 34.2)
- moved J4 0.30 mm to (131.8, 59.5)
- moved C1 0.22 mm to (137.1, 54.1)
- moved C4 0.20 mm to (140.6, 54.1)
Routing:
- net Net-(J4-Pad3): track 13.8 -> 14.3 mm
Other:
- board text added: "+3.3"
- board text added: "CS"
- board text added: "GND"
- board text added: "MISO"
- board text added: "MOSI"
- board text added: "RX"
- board text added: "SCK"
- board text added: "TX"
Changed lines of the file:
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@@
       (layerselection 0x00010fc_ffffffff)
       (disableapertmacros false)
-      (usegerberextensions false)
+      (usegerberextensions true)
       (usegerberattributes true)
-      (usegerberadvancedattributes true)
-      (creategerberjobfile true)
+      (usegerberadvancedattributes false)
+      (creategerberjobfile false)
       (svguseinch false)
       (svgprecision 6)
@@
       (psa4output false)
       (plotreference true)
-      (plotvalue true)
+      (plotvalue false)
       (plotinvisibletext false)
       (sketchpadsonfab false)
-      (subtractmaskfromsilk false)
+      (subtractmaskfromsilk true)
       (outputformat 1)
       (mirror false)
-      (drillshape 1)
+      (drillshape 0)
       (scaleselection 1)
-      (outputdirectory "")
+      (outputdirectory "gerbers/")
     )
   )
@@
   (net 24 "Net-(RN1-Pad5)")
   (footprint "MountingHole:MountingHole_3.2mm_M3" (layer "F.Cu")
-    (at 124.65 93)
+    (at 124.275 93.575)
     (descr "Mounting Hole 3.2mm, no annular, M3")
     (tags "mounting hole 3.2mm no annular m3")
@@
   )
   (footprint "G17C0900132EU:G17C0900132EU" (layer "F.Cu")
-    (at 131.933 59.317 -90)
+    (at 131.75 59.55 -90)
     (descr "G17C0900132EU-1")
     (tags "Capacitor")
@@
   )
   (footprint "MountingHole:MountingHole_3.2mm_M3" (layer "F.Cu")
-    (at 151.85 92.9)
+    (at 152.25 93.5)
     (descr "Mounting Hole 3.2mm, no annular, M3")
     (tags "mounting hole 3.2mm no annular m3")
@@
   )
   (footprint "MountingHole:MountingHole_3.2mm_M3" (layer "F.Cu")
-    (at 151.95 34.85)
+    (at 151.875 34.2)
     (descr "Mounting Hole 3.2mm, no annular, M3")
     (tags "mounting hole 3.2mm no annular m3")
@@
     (property "Sheetname" "")
     (attr smd)
-    (fp_text reference "C2" (at 0 -1.43 90) (layer "F.SilkS")
+    (fp_text reference "C2" (at -2.6295 -0.092 90) (layer "F.SilkS")
       (effects (font (size 1 1) (thickness 0.15)))
     )
@@
   )
   (footprint "Capacitor_SMD:C_0603_1608Metric_Pad1.08x0.95mm_HandSolder" (layer "F.Cu")
-    (at 137.0955 54.342 180)
+    (at 137.1125 54.125 180)
     (descr "Capacitor SMD 0603 (1608 Metric), square (rectangular) end terminal, IPC_7351 nominal with elongated pad for handsoldering. (Body size source: IPC-SM-782 page 76, https://www.pcb-3d.com/wordpress/wp-content/uploads/ipc-sm-782a_amendment_1_and_2.pdf), generated with kicad-footprint-generator")
     (tags "capacitor handsolder")
@@
     (property "Sheetname" "")
     (attr smd)
-    (fp_text reference "C1" (at 0 -1.43) (layer "F.SilkS")
+    (fp_text reference "C1" (at 2.5955 -0.008) (layer "F.SilkS")
       (effects (font (size 1 1) (thickness 0.15)))
     )
@@
     (property "Sheetname" "")
     (attr smd)
-    (fp_text reference "C5" (at 0 -1.43) (layer "F.SilkS")
+    (fp_text reference "C5" (at 2.6545 0.083) (layer "F.SilkS")
       (effects (font (size 1 1) (thickness 0.15)))
     )
@@
     (property "Sheetname" "")
     (attr smd)
-    (fp_text reference "C3" (at 0 -1.43 90) (layer "F.SilkS")
+    (fp_text reference "C3" (at 2.4955 -0.042 90) (layer "F.SilkS")
       (effects (font (size 1 1) (thickness 0.15)))
     )
@@
     (property "Sheetname" "")
     (attr smd)
-    (fp_text reference "U1" (at 0 -3.45) (layer "F.SilkS")
+    (fp_text reference "U1" (at -3.183 3.558) (layer "F.SilkS")
       (effects (font (size 1 1) (thickness 0.15)))
     )
@@
   )
   (footprint "MountingHole:MountingHole_3.2mm_M3" (layer "F.Cu")
-    (at 125.9 35.45)
+    (at 125 34.08)
     (descr "Mounting Hole 3.2mm, no annular, M3")
     (tags "mounting hole 3.2mm no annular m3")
@@
   )
   (footprint "Capacitor_SMD:C_0603_1608Metric_Pad1.08x0.95mm_HandSolder" (layer "F.Cu")
-    (at 140.5955 54.342 180)
+    (at 140.6025 54.14 180)
     (descr "Capacitor SMD 0603 (1608 Metric), square (rectangular) end terminal, IPC_7351 nominal with elongated pad for handsoldering. (Body size source: IPC-SM-782 page 76, https://www.pcb-3d.com/wordpress/wp-content/uploads/ipc-sm-782a_amendment_1_and_2.pdf), generated with kicad-footprint-generator")
     (tags "capacitor handsolder")
@@
     (property "Sheetname" "")
     (attr smd)
-    (fp_text reference "C4" (at 0 -1.43) (layer "F.SilkS")
+    (fp_text reference "C4" (at -2.6295 0.042) (layer "F.SilkS")
       (effects (font (size 1 1) (thickness 0.15)))
     )
@@
   (gr_line (start 155.45 96.55) (end 155.5 30.7) (layer "Edge.Cuts") (width 0.1))
   (gr_line (start 121 30.7) (end 121 63.5) (layer "Edge.Cuts") (width 0.1))
+  (gr_text "RX" (at 149.025 60.375) (layer "F.SilkS")
+    (effects (font (size 1 1) (thickness 0.15)))
+  )
+  (gr_text "+3.3" (at 150.1 53.35) (layer "F.SilkS")
+    (effects (font (size 1 1) (thickness 0.15)))
+  )
+  (gr_text "MISO" (at 148.3 74.275) (layer "F.SilkS")
+    (effects (font (size 1 1) (thickness 0.15)))
+  )
+  (gr_text "+3.3" (at 148.175 71.65) (layer "F.SilkS")
+    (effects (font (size 1 1) (thickness 0.15)))
+  )
+  (gr_text "SCK" (at 148.475 76.875) (layer "F.SilkS")
+    (effects (font (size 1 1) (thickness 0.15)))
+  )
+  (gr_text "GND" (at 148.725 84.25) (layer "F.SilkS")
+    (effects (font (size 1 1) (thickness 0.15)))
+  )
+  (gr_text "MOSI" (at 148.45 79.25) (layer "F.SilkS")
+    (effects (font (size 1 1) (thickness 0.15)))
+  )
+  (gr_text "CS" (at 148.9 81.95) (layer "F.SilkS")
+    (effects (font (size 1 1) (thickness 0.15)))
+  )
+  (gr_text "GND" (at 148.6 63.125) (layer "F.SilkS")
+    (effects (font (size 1 1) (thickness 0.15)))
+  )
+  (gr_text "TX" (at 149.175 57.95) (layer "F.SilkS")
+    (effects (font (size 1 1) (thickness 0.15)))
+  )
   (segment (start 138.8455 55.2295) (end 137.958 54.342) (width 0.25) (layer "F.Cu") (net 1))
   (segment (start 138.8455 55.817) (end 138.8455 55.2295) (width 0.25) (layer "F.Cu") (net 1))
@@
   (segment (start 131.933 56.545) (end 133.911 56.545) (width 0.25) (layer "F.Cu") (net 17))
   (segment (start 133.911 56.545) (end 133.911 56.602995) (width 0.25) (layer "F.Cu") (net 17))
-  (segment (start 131.183 57.817) (end 130.433 57.067) (width 0.25) (layer "F.Cu") (net 18))
-  (segment (start 131.47528 55.02472) (end 131.933 54.567) (width 0.25) (layer "F.Cu") (net 18))
-  (segment (start 130.433 57.067) (end 130.433 55.817) (width 0.25) (layer "F.Cu") (net 18))
-  (segment (start 133.433 57.817) (end 131.183 57.817) (width 0.25) (layer "F.Cu") (net 18))
+  (segment (start 131.75 54.005) (end 131.75 54.5) (width 0.25) (layer "F.Cu") (net 18))
+  (segment (start 133.966 58.1) (end 131.18 58.1) (width 0.25) (layer "F.Cu") (net 18))
+  (segment (start 136.233 60.367) (end 133.966 58.1) (width 0.25) (layer "F.Cu") (net 18))
+  (segment (start 138.8455 60.367) (end 136.233 60.367) (width 0.25) (layer "F.Cu") (net 18))
+  (segment (start 131.18 58.1) (end 130.433 57.353) (width 0.25) (layer "F.Cu") (net 18))
   (segment (start 131.933 54.567) (end 131.933 53.772) (width 0.25) (layer "F.Cu") (net 18))
-  (segment (start 133.683 57.817) (end 136.233 60.367) (width 0.25) (layer "F.Cu") (net 18))
-  (segment (start 131.22528 55.02472) (end 131.47528 55.02472) (width 0.25) (layer "F.Cu") (net 18))
-  (segment (start 138.8455 60.367) (end 136.233 60.367) (width 0.25) (layer "F.Cu") (net 18))
-  (segment (start 133.433 57.817) (end 133.683 57.817) (width 0.25) (layer "F.Cu") (net 18))
-  (segment (start 130.433 55.817) (end 131.22528 55.02472) (width 0.25) (layer "F.Cu") (net 18))
+  (segment (start 131.75 54.5) (end 131.11 55.14) (width 0.25) (layer "F.Cu") (net 18))
+  (segment (start 130.433 55.817) (end 131.11 55.14) (width 0.25) (layer "F.Cu") (net 18))
+  (segment (start 130.433 57.353) (end 130.433 55.817) (width 0.25) (layer "F.Cu") (net 18))
   (segment (start 127.683 51.567) (end 128.25 51) (width 0.25) (layer "F.Cu") (net 19))
   (segment (start 127.683 56.521) (end 127.683 51.567) (width 0.25) (layer "F.Cu") (net 19))
